Commit message: URDF Modified

File: turtlebot3_manipulation/turtlebot3_manipulation_description/urdf/open_manipulator_x.urdf.xacro (robot description, xacro)
@@ -94,5 +94,5 @@
     <parent link="link3"/>
     <child link="link4"/>
-    <origin xyz="0.024 0 0.128" rpy="0 ${pi/3} 0"/>
+    <origin xyz="0.024 0 0.128" rpy="0 ${pi/2} 0"/>
     <axis xyz="0 1 0"/>
     <limit velocity="4.8" effort="1" lower="${-pi*0.3}" upper="${pi*0.44}" />
@@ -100,10 +100,11 @@
   <!--  Link 4 -->
   <link name="link4">
-    <visual>
-      <origin xyz="0 0 0" rpy="0 0 0"/>
+      <visual>
+      <origin xyz="0 0 0.03" rpy="0 0 0"/>
       <geometry>
-        <mesh filename="package://turtlebot3_manipulation_description/meshes/chain_link4.stl" scale="0.001 0.001 0.001"/>
+        <box size="0.133 0.133 0.009"/>
+        <!-- <mesh filename="package://turtlebot3_description/meshes/bases/waffle_pi_base_for_open_manipulator.stl" scale="0.001 0.001 0.001"/> -->
       </geometry>
-      <material name="grey"/>
+      <material name="light_black"/>
     </visual>
     <collision>
@@ -121,70 +122,3 @@
     </inertial>
   </link>
-  <!--  Joint 4 -->
-  <joint name="joint4" type="revolute">
-    <parent link="link4"/>
-    <child link="link5"/>
-    <origin xyz="0.124 0.0 0.0" rpy="0 -${pi/3} 0"/>
-    <axis xyz="0 1 0"/>
-    <limit velocity="4.8" effort="1" lower="${-pi*0.57}" upper="${pi*0.65}" />
-  </joint>
-  <!--  Link 5 -->
-  <link name="link5">
-    <visual>
-      <origin xyz="0 0 0" rpy="0 0 0"/>
-      <geometry>
-        <mesh filename="package://turtlebot3_manipulation_description/meshes/chain_link5.stl" scale="0.001 0.001 0.001"/>
-      </geometry>
-      <material name="grey"/>
-    </visual>
-    <collision>
-      <origin xyz="0 0 0" rpy="0 0 0"/>
-      <geometry>
-        <mesh filename="package://turtlebot3_manipulation_description/meshes/chain_link5.stl" scale="0.001 0.001 0.001"/>
-      </geometry>
-    </collision>
-    <inertial>
-      <origin xyz="4.4206755e-02 3.6839985e-07 8.9142216e-03" />
-      <!-- <mass value="1.4327573e-01" />
-      <inertia ixx="8.0870749e-05" ixy="0.0" ixz="-1.0157896e-06"
-               iyy="7.5980465e-05" iyz="0.0"
-               izz="9.3127351e-05" /> -->
-      <mass value="1.0e-03" />
-      <inertia ixx="1.0e-03" ixy="0.0" ixz="0.0"
-               iyy="1.0e-03" iyz="0.0"
-               izz="1.0e-03" />
-    </inertial>
-  </link>
-  <!--  Gripper link -->
-  <link name="gripper_link">
-    <visual>
-      <origin xyz="0.064 0 0.064" rpy="0 0 0"/>
-      <geometry>
-        <box size="0.133 0.133 0.009"/>
-        <!-- <mesh filename="package://turtlebot3_description/meshes/bases/waffle_pi_base_for_open_manipulator.stl" scale="0.001 0.001 0.001"/> -->
-      </geometry>
-      <material name="light_black"/>
-    </visual>
-    <collision>
-      <origin xyz="-0.064 0 0.0045" rpy="0 0 0"/>
-      <geometry>
-        <box size="0.133 0.133 0.009"/>
-      </geometry>
-    </collision>
-    <inertial>
-      <origin xyz="0 0 0" />
-      <mass value="1.0e-03" />
-      <inertia ixx="1.0e-03" ixy="0.0" ixz="0.0"
-               iyy="1.0e-03" iyz="0.0"
-               izz="1.0e-03" />
-    </inertial>
-  </link>
-  <!--  Gripper joint -->
-  <joint name="gripper" type="prismatic">
-    <parent link="link5"/>
-    <child link="gripper_link"/>
-    <origin xyz="0.009 0 0.064" rpy="0 ${pi/2} 0"/>
-    <axis xyz="0 1 0"/>
-    <limit velocity="4.8" effort="1" lower="-0.010" upper="0.019" />
-  </joint>
 </robot>
