Commit message: Gripper Errors Modified, but Moveit doesn't work

File: turtlebot3_manipulation/turtlebot3_manipulation_description/urdf/open_manipulator_x.gazebo.xacro (robot description, xacro)
@@ -19,12 +19,4 @@
   <!-- Link3 -->
   <RefLink ref="link3"/>
-  <!-- Link4 -->
-  <RefLink ref="link4"/>
-  <!-- Link5 -->
-  <RefLink ref="link5"/>
-  <!-- gripper_link -->
-  <RefLink ref="gripper_link"/>
-  <!-- gripper_link_sub -->
-  <RefLink ref="gripper_link_sub"/>
   <!-- end effector link -->
   <gazebo reference="end_effector_link">
@@ -39,13 +31,3 @@
     </plugin>
   </gazebo>
-  <!--gazebo>
-    <! loading plugin: mimic joints works in gazebo now >
-    <plugin name="gazebo_gripper_ros_control" filename="libroboticsgroup_gazebo_mimic_joint_plugin.so">
-      <joint>gripper</joint>
-      <mimicJoint>gripper_sub</mimicJoint>
-      <multiplier>1.0</multiplier>
-      <offset>0.0</offset>
-      <hasPID>/gazebo_ros_control/pid_gains/gripper_sub</hasPID>
-    </plugin>
-  </gazebo>-->
 </robot>

File: turtlebot3_manipulation/turtlebot3_manipulation_description/urdf/open_manipulator_x.transmission.xacro (robot description, xacro)
@@ -33,9 +33,3 @@
   <!-- Transmission 3 -->
   <xacro:SimpleTransmissionPosition n="3" joint="joint3" />
-  <!-- Transmission 4 -->
-  <xacro:SimpleTransmissionPosition n="4" joint="joint4" />
-  <!-- Transmission 5 -->
-  <xacro:SimpleTransmissionEffort n="5" joint="gripper" />
-  <!-- Transmission 6 -->
-  <!-- xacro:SimpleTransmissionEffort n="6" joint="gripper_sub" /-->
 </robot>

Commit message: 200802

File: turtlebot3_manipulation/turtlebot3_manipulation_description/urdf/open_manipulator_x.gazebo.xacro (robot description, xacro)
@@ -19,4 +19,12 @@
   <!-- Link3 -->
   <RefLink ref="link3"/>
+  <!-- Link4 -->
+  <RefLink ref="link4"/>
+  <!-- Link5 -->
+  <RefLink ref="link5"/>
+  <!-- gripper_link -->
+  <RefLink ref="gripper_link"/>
+  <!-- gripper_link_sub -->
+  <RefLink ref="gripper_link_sub"/>
   <!-- end effector link -->
   <gazebo reference="end_effector_link">
@@ -31,3 +39,13 @@
     </plugin>
   </gazebo>
+  <!--gazebo>
+    <! loading plugin: mimic joints works in gazebo now >
+    <plugin name="gazebo_gripper_ros_control" filename="libroboticsgroup_gazebo_mimic_joint_plugin.so">
+      <joint>gripper</joint>
+      <mimicJoint>gripper_sub</mimicJoint>
+      <multiplier>1.0</multiplier>
+      <offset>0.0</offset>
+      <hasPID>/gazebo_ros_control/pid_gains/gripper_sub</hasPID>
+    </plugin>
+  </gazebo>-->
 </robot>

File: turtlebot3_manipulation/turtlebot3_manipulation_description/urdf/open_manipulator_x.transmission.xacro (robot description, xacro)
@@ -33,3 +33,5 @@
   <!-- Transmission 3 -->
   <xacro:SimpleTransmissionPosition n="3" joint="joint3" />
+  <!-- Transmission 6 -->
+  <!-- xacro:SimpleTransmissionEffort n="6" joint="gripper_sub" /-->
 </robot>
