Commit message: Waypoints Confirmed

File: turtlebot3/turtlebot3_description/urdf/turtlebot3_waffle_pi_for_open_manipulator.urdf.xacro (robot description, xacro)
@@ -196,5 +196,6 @@
   </link>
   <joint name="camera_joint" type="fixed">
-    <origin xyz="0.073 -0.011 0.084" rpy="0 0 0"/>
+    <!-- origin xyz="0.073 -0.011 0.084" rpy="0 0 0"/ -->
+    <origin xyz="0.045 0.0 0.009" rpy="0 0 0"/>
     <parent link="base_link"/>
     <child link="camera_link"/>
@@ -202,9 +203,15 @@
   <link name="camera_link">
     <collision>
-      <origin xyz="0.005 0.011 0.013" rpy="0 0 0"/>
+      <origin xyz="0.005 0.0 0.013" rpy="0 0 0"/>
       <geometry>
         <box size="0.015 0.030 0.027"/>
       </geometry>
     </collision>
+    <visual>
+      <origin xyz="0.005 0.0 0.013" rpy="0 0 0"/>
+      <geometry>
+        <box size="0.015 0.030 0.027"/>
+      </geometry>
+    </visual>
   </link>
   <joint name="camera_rgb_joint" type="fixed">

File: turtlebot3_manipulation/turtlebot3_manipulation_description/urdf/open_manipulator_x.urdf.xacro (robot description, xacro)
@@ -14,10 +14,10 @@
       <material name="grey"/>
     </visual>
-    <collision>
+    <!-- collision>
       <origin xyz="0 0 0" rpy="0 0 0"/>
       <geometry>
         <mesh filename="package://turtlebot3_manipulation_description/meshes/chain_link1.stl" scale="0.001 0.001 0.001"/>
       </geometry>
-    </collision>
+    </collision -->
      <inertial>
       <origin xyz="3.0876154e-04 0.0000000e+00 -1.2176461e-04" />
@@ -45,10 +45,10 @@
       <material name="grey"/>
     </visual>
-    <collision>
+    <!-- collision>
       <origin xyz="0 0 0.018" rpy="0 0 0"/>
       <geometry>
         <mesh filename="package://turtlebot3_manipulation_description/meshes/chain_link2.stl" scale="0.001 0.001 0.001"/>
       </geometry>
-    </collision>
+    </collision -->
      <inertial>
       <origin xyz="-3.0184870e-04 5.4043684e-04 ${0.018 + 2.9433464e-02}" />
@@ -76,10 +76,10 @@
       <material name="grey"/>
     </visual>
-    <collision>
+    <!-- collision>
       <origin xyz="0 0 0" rpy="0 0 0"/>
       <geometry>
         <mesh filename="package://turtlebot3_manipulation_description/meshes/chain_link3.stl" scale="0.001 0.001 0.001"/>
       </geometry>
-    </collision>
+    </collision -->
      <inertial>
       <origin xyz="1.0308393e-02 3.7743363e-04 1.0170197e-01" />
