Commit message: 200818_1

File: turtlebot3/turtlebot3_description/urdf/turtlebot3_waffle_pi_for_open_manipulator.gazebo.xacro (robot description, xacro)
@@ -3,4 +3,6 @@
   <xacro:arg name="laser_visual"  default="false"/>
   <xacro:arg name="camera_visual" default="false"/>
+  <xacro:arg name="sub_camera_visual1" default="false"/>
+  <xacro:arg name="sub_camera_visual2" default="false"/>
   <xacro:arg name="imu_visual"    default="false"/>
   <gazebo reference="base_link">
@@ -135,4 +137,5 @@
   </gazebo>
 <!--link : https://www.raspberrypi.org/documentation/hardware/camera/-->
+<!-- main camera -->
   <gazebo reference="camera_rgb_frame">
     <sensor type="camera" name="Pi Camera">
@@ -167,3 +170,69 @@
     </sensor>
   </gazebo>
+<!-- sub cam 1 -->
+  <gazebo reference="sub_camera_rgb_frame1">
+    <sensor type="camera" name="sub Pi Camera1">
+      <always_on>true</always_on>
+      <visualize>$(arg sub_camera_visual1)</visualize>
+      <camera>
+          <horizontal_fov>1.085595</horizontal_fov>
+          <image>
+              <width>640</width>
+              <height>480</height>
+              <format>R8G8B8</format>
+          </image>
+          <clip>
+              <near>0.03</near>
+              <far>100</far>
+          </clip>
+      </camera>
+      <plugin name="sub_camera_controller1" filename="libgazebo_ros_camera.so">
+        <alwaysOn>true</alwaysOn>
+        <updateRate>30.0</updateRate>
+        <cameraName>sub_camera1</cameraName>
+        <frameName>sub_camera_rgb_optical_frame1</frameName>
+        <imageTopicName>rgb/image_raw</imageTopicName>
+        <cameraInfoTopicName>rgb/camera_info</cameraInfoTopicName>
+        <hackBaseline>0.07</hackBaseline>
+        <distortionK1>0.0</distortionK1>
+        <distortionK2>0.0</distortionK2>
+        <distortionK3>0.0</distortionK3>
+        <distortionT1>0.0</distortionT1>
+        <distortionT2>0.0</distortionT2>
+      </plugin>
+    </sensor>
+  </gazebo>
+  <!-- sub cam 2 -->
+  <gazebo reference="sub_camera_rgb_frame2">
+    <sensor type="camera" name="sub Pi Camera2">
+      <always_on>true</always_on>
+      <visualize>$(arg sub_camera_visual2)</visualize>
+      <camera>
+          <horizontal_fov>1.085595</horizontal_fov>
+          <image>
+              <width>640</width>
+              <height>480</height>
+              <format>R8G8B8</format>
+          </image>
+          <clip>
+              <near>0.03</near>
+              <far>100</far>
+          </clip>
+      </camera>
+      <plugin name="sub_camera_controller2" filename="libgazebo_ros_camera.so">
+        <alwaysOn>true</alwaysOn>
+        <updateRate>30.0</updateRate>
+        <cameraName>sub_camera2</cameraName>
+        <frameName>sub_camera_rgb_optical_frame2</frameName>
+        <imageTopicName>rgb/image_raw</imageTopicName>
+        <cameraInfoTopicName>rgb/camera_info</cameraInfoTopicName>
+        <hackBaseline>0.07</hackBaseline>
+        <distortionK1>0.0</distortionK1>
+        <distortionK2>0.0</distortionK2>
+        <distortionK3>0.0</distortionK3>
+        <distortionT1>0.0</distortionT1>
+        <distortionT2>0.0</distortionT2>
+      </plugin>
+    </sensor>
+  </gazebo>
 </robot>

File: turtlebot3/turtlebot3_description/urdf/turtlebot3_waffle_pi_for_open_manipulator.urdf.xacro (robot description, xacro)
@@ -195,7 +195,7 @@
     </inertial>
   </link>
+  <!-- Main Camera -->
   <joint name="camera_joint" type="fixed">
-    <!-- origin xyz="0.073 -0.011 0.084" rpy="0 0 0"/ -->
-    <origin xyz="0.045 0.0 0.009" rpy="0 0 0"/>
+    <origin xyz="0.045 0.0 0.009" rpy="0 -${pi/6} 0"/>
     <parent link="base_link"/>
     <child link="camera_link"/>
@@ -227,3 +227,68 @@
   </joint>
   <link name="camera_rgb_optical_frame"/>
+  <!-- Sub Camera 1 -->
+  <joint name="sub_camera_joint1" type="fixed">
+    <!-- origin xyz="0.045 0.0 0.009" rpy="0 0 0"/ -->
+    <origin xyz="-0.174 0.10 0.009" rpy="0 -${pi/6} ${pi}"/>
+    <parent link="base_link"/>
+    <child link="sub_camera_link1"/>
+  </joint>
+  <link name="sub_camera_link1">
+    <collision>
+      <origin xyz="0.005 0.0 0.013" rpy="0 0 0"/>
+      <geometry>
+        <box size="0.015 0.030 0.027"/>
+      </geometry>
+    </collision>
+    <visual>
+      <origin xyz="0.005 0.0 0.013" rpy="0 0 0"/>
+      <geometry>
+        <box size="0.015 0.030 0.027"/>
+      </geometry>
+    </visual>
+  </link>
+  <joint name="sub_camera_rgb_joint1" type="fixed">
+    <origin xyz="0.003 0.011 0.009" rpy="0 0 0"/>
+    <parent link="sub_camera_link1"/>
+    <child link="sub_camera_rgb_frame1"/>
+  </joint>
+  <link name="sub_camera_rgb_frame1"/>
+  <joint name="sub_camera_rgb_optical_joint1" type="fixed">
+    <origin xyz="0 0 0" rpy="-1.57 0 -1.57"/>
+    <parent link="sub_camera_rgb_frame1"/>
+    <child link="sub_camera_rgb_optical_frame1"/>
+  </joint>
+  <link name="sub_camera_rgb_optical_frame1"/>
+  <!-- Sub Camera 2 -->
+    <joint name="sub_camera_joint2" type="fixed">
+    <origin xyz="-0.174 -0.10 0.009" rpy="0 -${pi/6} ${pi}"/>
+    <parent link="base_link"/>
+    <child link="sub_camera_link2"/>
+  </joint>
+  <link name="sub_camera_link2">
+    <collision>
+      <origin xyz="0.005 0.0 0.013" rpy="0 0 0"/>
+      <geometry>
+        <box size="0.015 0.030 0.027"/>
+      </geometry>
+    </collision>
+    <visual>
+      <origin xyz="0.005 0.0 0.013" rpy="0 0 0"/>
+      <geometry>
+        <box size="0.015 0.030 0.027"/>
+      </geometry>
+    </visual>
+  </link>
+  <joint name="sub_camera_rgb_joint2" type="fixed">
+    <origin xyz="0.003 0.011 0.009" rpy="0 0 0"/>
+    <parent link="sub_camera_link2"/>
+    <child link="sub_camera_rgb_frame2"/>
+  </joint>
+  <link name="sub_camera_rgb_frame2"/>
+  <joint name="sub_camera_rgb_optical_joint2" type="fixed">
+    <origin xyz="0 0 0" rpy="-1.57 0 -1.57"/>
+    <parent link="sub_camera_rgb_frame2"/>
+    <child link="sub_camera_rgb_optical_frame2"/>
+  </joint>
+  <link name="sub_camera_rgb_optical_frame2"/>
 </robot>

Commit message: 200904_2104

File: turtlebot3/turtlebot3_description/urdf/turtlebot3_waffle_pi_for_open_manipulator.gazebo.xacro (robot description, xacro)
@@ -5,4 +5,5 @@
   <xacro:arg name="sub_camera_visual1" default="false"/>
   <xacro:arg name="sub_camera_visual2" default="false"/>
+  <xacro:arg name="manipulator_cam_visual" default="false"/>
   <xacro:arg name="imu_visual"    default="false"/>
   <gazebo reference="base_link">
@@ -236,3 +237,36 @@
     </sensor>
   </gazebo>
+  <!-- manipulator cam -->
+  <gazebo reference="manipulator_cam_rgb_frame">
+    <sensor type="camera" name="sub Pi Camera2">
+      <always_on>true</always_on>
+      <visualize>$(arg manipulator_cam_visual)</visualize>
+      <camera>
+          <horizontal_fov>1.085595</horizontal_fov>
+          <image>
+              <width>640</width>
+              <height>480</height>
+              <format>R8G8B8</format>
+          </image>
+          <clip>
+              <near>0.03</near>
+              <far>100</far>
+          </clip>
+      </camera>
+      <plugin name="manipulator_cam_controller" filename="libgazebo_ros_camera.so">
+        <alwaysOn>true</alwaysOn>
+        <updateRate>30.0</updateRate>
+        <cameraName>manipulator_cam</cameraName>
+        <frameName>manipulator_cam_rgb_optical_frame</frameName>
+        <imageTopicName>rgb/image_raw</imageTopicName>
+        <cameraInfoTopicName>rgb/camera_info</cameraInfoTopicName>
+        <hackBaseline>0.07</hackBaseline>
+        <distortionK1>0.0</distortionK1>
+        <distortionK2>0.0</distortionK2>
+        <distortionK3>0.0</distortionK3>
+        <distortionT1>0.0</distortionT1>
+        <distortionT2>0.0</distortionT2>
+      </plugin>
+    </sensor>
+  </gazebo>
 </robot>

File: turtlebot3_manipulation/turtlebot3_manipulation_description/urdf/open_manipulator_x.urdf.xacro (robot description, xacro)
@@ -63,5 +63,5 @@
     <parent link="link2"/>
     <child link="link3"/>
-    <origin xyz="0.0 0.0 0.058" rpy="0 -${pi/2} 0"/>
+    <origin xyz="0.0 0.0 0.058" rpy="0 -${pi/2 + pi/6} 0"/>
     <axis xyz="0 1 0"/>
     <limit velocity="4.8" effort="1" lower="${-pi*0.57}" upper="${pi*0.5}" />
@@ -94,5 +94,5 @@
     <parent link="link3"/>
     <child link="link4"/>
-    <origin xyz="0.024 0 0.128" rpy="0 ${pi/2} 0"/>
+    <origin xyz="0.024 0 0.128" rpy="0 ${pi/2 + pi/6} 0"/>
     <axis xyz="0 1 0"/>
     <limit velocity="4.8" effort="1" lower="${-pi*0.3}" upper="${pi*0.44}" />

File: turtlebot3_manipulation/turtlebot3_manipulation_description/urdf/turtlebot3_manipulation_robot.urdf.xacro (robot description, xacro)
@@ -11,3 +11,35 @@
     <child link="link1"/>
   </joint>
+  <!-- Manipulator Camera -->
+  <joint name="manipulator_cam_joint" type="fixed">
+    <origin xyz="-0.08 0 0.025" rpy="0 -${pi/2} ${pi}"/>
+    <parent link="link4"/>
+    <child link="manipulator_cam"/>
+  </joint>
+  <link name="manipulator_cam">
+    <collision>
+      <origin xyz="0.0 0.0 0.0" rpy="0 0 0"/>
+      <geometry>
+        <box size="0.015 0.030 0.027"/>
+      </geometry>
+    </collision>
+    <visual>
+      <origin xyz="0.0 0.0 0.0" rpy="0 0 0"/>
+      <geometry>
+        <box size="0.015 0.030 0.027"/>
+      </geometry>
+    </visual>
+  </link>
+  <joint name="manipulator_cam_rgb_joint" type="fixed">
+    <origin xyz="0.003 0.011 0.009" rpy="0 0 0"/>
+    <parent link="manipulator_cam"/>
+    <child link="manipulator_cam_rgb_frame"/>
+  </joint>
+  <link name="manipulator_cam_rgb_frame"/>
+  <joint name="manipulator_cam_rgb_optical_joint" type="fixed">
+    <origin xyz="0 0 0" rpy="-1.57 0 -1.57"/>
+    <parent link="manipulator_cam_rgb_frame"/>
+    <child link="manipulator_cam_rgb_optical_frame"/>
+  </joint>
+  <link name="manipulator_cam_rgb_optical_frame"/>
 </robot>
